File: Step-by-Step-DAQ/DAQ1.brd (EAGLE design)
At the start: 106.8 x 75 mm, 28 parts, among them IC1 PIC18F4550_40, IC2 7805T, Q1 20MHz, X1 PN61729-S

Commit message: Clase #2
Parts:
- moved IC1 83.4 mm to (-34.4, 75.8)
Connections:
- new net GND: C1.1, C2.1, C4.-, IC2.2, J1.1
- new net N$1: C4.+, IC2.3, J1.3
- new net N$2: C5.1, IC2.1
- new net X1: C1.2, IC1.13, Q1.1
- new net X2: C2.2, IC1.14, Q1.2
Changed lines of the file:
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@@
 <attribute name="VALUE" x="-112.1791" y="10.414" size="1.27" layer="27" font="vector" ratio="16" rot="R180"/>
 </element>
-<element name="IC1" library="microchip" package="DIL40" value="PIC18F4550_40" x="-117.6782" y="78.2574" rot="R270">
-<attribute name="OC_NEWARK" value="74K8623" x="-117.6782" y="78.2574" size="1.778" layer="27" rot="R270" display="off"/>
-<attribute name="MPN" value="PIC18F4550-I/P" x="-117.6782" y="78.2574" size="1.778" layer="27" rot="R270" display="off"/>
-<attribute name="MF" value="MICROCHIP" x="-117.6782" y="78.2574" size="1.778" layer="27" rot="R270" display="off"/>
-<attribute name="OC_FARNELL" value="9321357" x="-117.6782" y="78.2574" size="1.778" layer="27" rot="R270" display="off"/>
+<element name="IC1" library="microchip" package="DIL40" value="PIC18F4550_40" x="-34.3535" y="75.819" rot="R270">
+<attribute name="OC_NEWARK" value="74K8623" x="-34.3535" y="75.819" size="1.778" layer="27" rot="R270" display="off"/>
+<attribute name="MPN" value="PIC18F4550-I/P" x="-34.3535" y="75.819" size="1.778" layer="27" rot="R270" display="off"/>
+<attribute name="MF" value="MICROCHIP" x="-34.3535" y="75.819" size="1.778" layer="27" rot="R270" display="off"/>
+<attribute name="OC_FARNELL" value="9321357" x="-34.3535" y="75.819" size="1.778" layer="27" rot="R270" display="off"/>
 </element>
 <element name="LED1" library="led" package="LED3MM" value="RED" x="-100.9904" y="43.7261" smashed="yes" rot="MR0">
@@
 <contactref element="IC1" pad="12"/>
 <contactref element="IC1" pad="31"/>
-<wire x1="-110.0582" y1="79.5274" x2="-125.2982" y2="74.4474" width="0" layer="19" extent="1-1"/>
+<wire x1="-41.9735" y1="72.009" x2="-26.7335" y2="77.089" width="0" layer="19" extent="1-1"/>
 </signal>
 <signal name="VDD">
 <contactref element="IC1" pad="11"/>
 <contactref element="IC1" pad="32"/>
-<wire x1="-110.0582" y1="82.0674" x2="-125.2982" y2="76.9874" width="0" layer="19" extent="1-1"/>
+<wire x1="-41.9735" y1="74.549" x2="-26.7335" y2="79.629" width="0" layer="19" extent="1-1"/>
 </signal>
 <signal name="N$4">
 <contactref element="," pad="1"/>
 </signal>
+<signal name="N$1">
+<contactref element="J1" pad="3"/>
+<contactref element="C4" pad="+"/>
+<contactref element="IC2" pad="3"/>
+<wire x1="-138.6332" y1="55.1561" x2="-124.8918" y2="40.4904" width="0" layer="19" extent="1-1"/>
+<wire x1="-85.3059" y1="18.923" x2="-124.8918" y2="40.4904" width="0" layer="19" extent="1-1"/>
+</signal>
+<signal name="GND">
+<contactref element="J1" pad="1"/>
+<contactref element="C4" pad="-"/>
+<contactref element="IC2" pad="2"/>
+<contactref element="C1" pad="1"/>
+<contactref element="C2" pad="1"/>
+<wire x1="-105.2576" y1="10.9855" x2="-113.7031" y2="11.557" width="0" layer="19" extent="1-1"/>
+<wire x1="-85.3059" y1="21.463" x2="-105.2576" y2="10.9855" width="0" layer="19" extent="1-1"/>
+<wire x1="-124.8918" y1="34.4904" x2="-113.7031" y2="11.557" width="0" layer="19" extent="1-1"/>
+<wire x1="-136.0932" y1="55.1561" x2="-124.8918" y2="34.4904" width="0" layer="19" extent="1-1"/>
+</signal>
+<signal name="X1">
+<contactref element="C1" pad="2"/>
+<contactref element="Q1" pad="1"/>
+<contactref element="IC1" pad="13"/>
+<wire x1="-72.0725" y1="18.6436" x2="-105.2576" y2="13.5255" width="0" layer="19" extent="1-1"/>
+<wire x1="-41.9735" y1="69.469" x2="-72.0725" y2="18.6436" width="0" layer="19" extent="1-1"/>
+</signal>
+<signal name="X2">
+<contactref element="IC1" pad="14"/>
+<contactref element="Q1" pad="2"/>
+<contactref element="C2" pad="2"/>
+<wire x1="-66.9925" y1="18.6436" x2="-113.7031" y2="14.097" width="0" layer="19" extent="1-1"/>
+<wire x1="-41.9735" y1="66.929" x2="-66.9925" y2="18.6436" width="0" layer="19" extent="1-1"/>
+</signal>
+<signal name="N$2">
+<contactref element="IC2" pad="1"/>
+<contactref element="C5" pad="1"/>
+<wire x1="-97.5487" y1="27.4701" x2="-133.5532" y2="55.1561" width="0" layer="19" extent="1-1"/>
+</signal>
 </signals>
